File: Hardware/Nodeboard/OECOC_controlbord.brd (EAGLE design)
At the start: 160 x 100 mm, 12 parts, among them IC1 DS2405, IC2 DS2405, U1 ESP32-DEVKITC-32D

Commit message: add buzzer
Parts:
- added SG1: B/C11S, buzzer:B/C11S
Connections:
- new net N$11: SG1.1, U1.10
- net GND: now also SG1.2
Changed lines of the file:
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@@
 <attribute name="VALUE" x="-121.6406" y="-4.445" size="1.27" layer="27" ratio="10"/>
+</element>
+<element name="SG1" library="buzzer" library_urn="urn:adsk.eagle:library:113" package="B/C11S" package3d_urn="urn:adsk.eagle:package:5277/1" value="B/C11S" x="-116.84" y="-10.16" smashed="yes">
+<attribute name="MF" value="" x="-116.84" y="-10.16" size="1.778" layer="27" display="off"/>
+<attribute name="MPN" value="" x="-116.84" y="-10.16" size="1.778" layer="27" display="off"/>
+<attribute name="NAME" x="-124.333" y="-7.239" size="1.27" layer="25" ratio="10"/>
+<attribute name="OC_FARNELL" value="unknown" x="-116.84" y="-10.16" size="1.778" layer="27" display="off"/>
+<attribute name="OC_NEWARK" value="unknown" x="-116.84" y="-10.16" size="1.778" layer="27" display="off"/>
+<attribute name="POPULARITY" value="2" x="-116.84" y="-10.16" size="1.778" layer="27" display="off"/>
+<attribute name="VALUE" x="-119.38" y="-13.97" size="1.27" layer="27" ratio="10"/>
 </element>
 </elements>
@@
 <contactref element="S2" pad="2"/>
 <contactref element="U$6" pad="8"/>
+<contactref element="SG1" pad="2"/>
 <wire x1="-22.86" y1="179.07" x2="-20.32" y2="179.07" width="0" layer="19" extent="1-1"/>
 <wire x1="-20.8" y1="168.91" x2="-20.32" y2="179.07" width="0" layer="19" extent="1-1"/>
@@
 <wire x1="-72.39" y1="35" x2="-72.39" y2="50.24" width="0" layer="19" extent="1-1"/>
 <wire x1="-97.79" y1="17.22" x2="-72.39" y2="35" width="0" layer="19" extent="1-1"/>
+<wire x1="-113.0808" y1="-10.16" x2="-97.79" y2="17.22" width="0" layer="19" extent="1-1"/>
 </signal>
 <signal name="+5V">
@@
 <wire x1="-97.79" y1="19.76" x2="-72.87" y2="168.91" width="0" layer="19" extent="1-1"/>
 </signal>
+<signal name="N$11">
+<contactref element="SG1" pad="1"/>
+<contactref element="U1" pad="10"/>
+<wire x1="-97.79" y1="27.38" x2="-120.5992" y2="-10.16" width="0" layer="19" extent="1-1"/>
+</signal>
 </signals>

Commit message: changed pins relay
Connections:
- net N$2: now also U1.12; no longer U1.32
- net N$7: now also U1.15; no longer U1.34
Changed lines of the file:
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@@
 <wire x1="-97.79" y1="4.52" x2="-17.78" y2="80.645" width="0" layer="19" extent="1-1"/>
-</signal>
-<signal name="N$2">
-<contactref element="U1" pad="32"/>
-<contactref element="U$1" pad="J1.4"/>
-<wire x1="-17.78" y1="73.025" x2="-72.39" y2="19.76" width="0" layer="19" extent="1-1"/>
 </signal>
 <signal name="N$3">
@@
 </signal>
 <signal name="N$7">
-<contactref element="U1" pad="34"/>
 <contactref element="U$1" pad="J1.3"/>
-<wire x1="-17.78" y1="75.565" x2="-72.39" y2="14.68" width="0" layer="19" extent="1-1"/>
+<contactref element="U1" pad="15"/>
+<wire x1="-17.78" y1="75.565" x2="-97.79" y2="14.68" width="0" layer="19" extent="1-1"/>
 </signal>
 <signal name="N$8">
@@
 <wire x1="-97.79" y1="27.38" x2="-120.5992" y2="-10.16" width="0" layer="19" extent="1-1"/>
 </signal>
+<signal name="N$2">
+<contactref element="U$1" pad="J1.4"/>
+<contactref element="U1" pad="12"/>
+<wire x1="-17.78" y1="73.025" x2="-97.79" y2="22.3" width="0" layer="19" extent="1-1"/>
+</signal>
 </signals>

Commit message: changed pin relay and reeds
Connections:
- net N$14: now also U1.12; no longer U1.13
- net N$2: now also U1.13; no longer U1.12
Changed lines of the file:
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@@
 <contactref element="S2" pad="1"/>
 <contactref element="U$6" pad="7"/>
-<contactref element="U1" pad="13"/>
+<contactref element="U1" pad="12"/>
 <wire x1="-72.87" y1="168.91" x2="-77.47" y2="179.07" width="0" layer="19" extent="1-1"/>
-<wire x1="-97.79" y1="19.76" x2="-72.87" y2="168.91" width="0" layer="19" extent="1-1"/>
+<wire x1="-97.79" y1="22.3" x2="-72.87" y2="168.91" width="0" layer="19" extent="1-1"/>
 </signal>
 <signal name="N$11">
@@
 <signal name="N$2">
 <contactref element="U$1" pad="J1.4"/>
-<contactref element="U1" pad="12"/>
-<wire x1="-17.78" y1="73.025" x2="-97.79" y2="22.3" width="0" layer="19" extent="1-1"/>
+<contactref element="U1" pad="13"/>
+<wire x1="-17.78" y1="73.025" x2="-97.79" y2="19.76" width="0" layer="19" extent="1-1"/>
 </signal>
 </signals>

Commit message: edit pins relay
Connections:
- net N$2: now also U1.9; no longer U1.13
Changed lines of the file:
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@@
 <signal name="N$2">
 <contactref element="U$1" pad="J1.4"/>
-<contactref element="U1" pad="13"/>
-<wire x1="-17.78" y1="73.025" x2="-97.79" y2="19.76" width="0" layer="19" extent="1-1"/>
+<contactref element="U1" pad="9"/>
+<wire x1="-17.78" y1="73.025" x2="-97.79" y2="29.92" width="0" layer="19" extent="1-1"/>
 </signal>
 </signals>

Commit message: add extra connectors
Parts:
- added H1, H2, H3, H4: MOUNT-PAD-ROUND3.2, holes:3,2-PAD
- added U$7, U$8: PHOENIXCONTACT_PINSTRIP, Personal:HDRV8W150P500_1X8_2488X140X1204B
- moved U$1 283.2 mm to (238.8, 34.3), turned to 180 degrees
- moved S2 251.0 mm to (47.0, -45.7), flipped to the bottom, turned to 180 degrees
- moved U$5 243.4 mm to (85.1, -20.3), turned to 270 degrees
- moved S1 230.7 mm to (16.5, -45.7), turned to 180 degrees
- moved IC1 229.4 mm to (16.5, -14.0), turned to 180 degrees
- moved U$2 212.5 mm to (63.5, -20.3), turned to 270 degrees
- moved U$6 201.2 mm to (14.0, 5.08)
- moved IC2 198.7 mm to (29.2, -14.0)
- moved U$3 194.8 mm to (54.6, 5.08)
- moved R1 151.8 mm to (25.4, 41.9), turned to 180 degrees
- moved U1 138.7 mm to (52.1, 50.8)
- moved U$4 132.0 mm to (-47.0, 24.1)
- moved SG1 89.9 mm to (-50.8, 50.8), turned to 180 degrees
Connections:
- new net VCC: U$4.1
- net +5V: now also U$8.5, U$8.7; no longer U$4.1
- net GND: now also H1.B3,2, H2.B3,2, H3.B3,2, H4.B3,2, U$8.2, U$8.4, U$8.6, U$8.8
- net N$1: now also U$8.3
- net N$11: now also U$8.1
- net N$2: now also U$7.6
- net N$3: now also U$7.5
- net N$4: now also U$7.4
- net N$5: now also U$7.3
- net N$6: now also U$7.8
- net N$7: now also U$7.7
- net N$8: now also U$7.2
- net N$9: now also U$7.1
Other:
- board size 160 x 100 mm -> 100 x 80 mm

Commit message: add pcb layout
Parts:
- moved S2 123.3 mm to (-22.9, 55.9), turned to 90 degrees
- moved U$4 118.1 mm to (29.2, 114.3), turned to 270 degrees
- moved S1 111.4 mm to (-29.2, 55.9), turned to 90 degrees
- moved U$8 106.2 mm to (31.8, 55.0), turned to 0 degrees
- moved SG1 80.0 mm to (14.0, 97.8), turned to 0 degrees
- moved U$1 75.1 mm to (163.8, 39.4), turned to 0 degrees
- moved IC2 63.8 mm to (-25.4, 19.1), turned to 270 degrees
- moved IC1 59.3 mm to (-25.4, 27.9), turned to 270 degrees
- moved U$7 51.2 mm to (90.0, 15.2), turned to 90 degrees
- moved U$2 25.4 mm to (38.1, -20.3)
- moved U$5 24.1 mm to (61.0, -20.3)
- moved R1 23.7 mm to (19.1, 19.1), turned to 270 degrees
- moved U$3 23.4 mm to (31.8, 10.0)
- moved U1 18.2 mm to (48.3, 33.0), turned to 90 degrees
- moved H4 14.9 mm to (95.0, 60.1)
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Connections:
- net N$10 renamed REED_2
- net N$11 renamed BUZZER
- net N$13 renamed DS18B20
- net N$14 renamed REED_1
- net N$2 renamed IN6
- net N$3 renamed IN5
- net N$4 renamed IN4
- net N$5 renamed IN3
- net N$6 renamed IN8
- net N$7 renamed IN7
- net N$8 renamed IN2
- net N$9 renamed IN1
Routing:
- added copper zone on layer 1, net GND
- added copper zone on layer 16, net GND
Other:
- board size 100 x 80 mm -> 100 x 65 mm
