File: Hardware/Nodeboard/OECOC_controlbord.sch (EAGLE design)
At the start: 13 parts, among them IC1 DS2405, IC2 DS2405, U1 ESP32-DEVKITC-32D

Commit message: add extra connectors
Parts:
- added H1, H2, H3, H4: MOUNT-PAD-ROUND3.2, holes:MOUNT-PAD-ROUND3.2
- added U$7, U$8: PHOENIXCONTACT_PINSTRIP, Personal:PHOENIXCONTACT_PINSTRIP
Connections:
- net +5V: now also U$8.5, U$8.7; no longer U$4.VCC
- net GND: now also H1.MOUNT, H2.MOUNT, H3.MOUNT, H4.MOUNT, U$8.2, U$8.4, U$8.6, U$8.8
- net N$1: now also U$8.3
- net N$11: now also U$8.1
- net N$2: now also U$7.6
- net N$3: now also U$7.5
- net N$4: now also U$7.4
- net N$5: now also U$7.3
- net N$6: now also U$7.8
- net N$7: now also U$7.7
- net N$8: now also U$7.2
- net N$9: now also U$7.1
Other:
- moved on the sheet: SG1, U$1, U$4

Commit message: add pcb layout
Connections:
- net N$10 renamed REED_2
- net N$11 renamed BUZZER
- net N$13 renamed DS18B20
- net N$14 renamed REED_1
- net N$2 renamed IN6
- net N$3 renamed IN5
- net N$4 renamed IN4
- net N$5 renamed IN3
- net N$6 renamed IN8
- net N$7 renamed IN7
- net N$8 renamed IN2
- net N$9 renamed IN1
Changed lines of the file:
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@@
 <attribute name="VALUE" x="23.114" y="7.6962" size="1.778" layer="96"/>
 </instance>
-<instance part="U$7" gate="G$1" x="335.28" y="161.29" smashed="yes"/>
+<instance part="U$7" gate="G$1" x="331.47" y="161.29" smashed="yes"/>
 <instance part="U$8" gate="G$1" x="269.24" y="236.22" smashed="yes"/>
 <instance part="G5" gate="G$1" x="256.54" y="229.87" smashed="yes">
@@
 </segment>
 </net>
-<net name="N$3" class="0">
+<net name="IN5" class="0">
 <segment>
 <pinref part="U1" gate="G$1" pin="IO16"/>
@@
 <wire x1="317.5" y1="170.18" x2="317.5" y2="171.45" width="0.1524" layer="91"/>
 <pinref part="U$1" gate="G$1" pin="IN5"/>
-<wire x1="346.71" y1="171.45" x2="340.36" y2="171.45" width="0.1524" layer="91"/>
+<wire x1="346.71" y1="171.45" x2="336.55" y2="171.45" width="0.1524" layer="91"/>
 <pinref part="U$7" gate="G$1" pin="5"/>
-<wire x1="340.36" y1="171.45" x2="317.5" y2="171.45" width="0.1524" layer="91"/>
-<junction x="340.36" y="171.45"/>
-</segment>
-</net>
-<net name="N$4" class="0">
+<wire x1="336.55" y1="171.45" x2="317.5" y2="171.45" width="0.1524" layer="91"/>
+<junction x="336.55" y="171.45"/>
+<label x="337.82" y="171.45" size="1.778" layer="95"/>
+</segment>
+</net>
+<net name="IN4" class="0">
 <segment>
 <pinref part="U1" gate="G$1" pin="IO17"/>
@@
 <pinref part="U$1" gate="G$1" pin="IN4"/>
 <wire x1="256.54" y1="172.72" x2="256.54" y2="173.99" width="0.1524" layer="91"/>
-<wire x1="256.54" y1="173.99" x2="340.36" y2="173.99" width="0.1524" layer="91"/>
+<wire x1="256.54" y1="173.99" x2="336.55" y2="173.99" width="0.1524" layer="91"/>
 <pinref part="U$7" gate="G$1" pin="4"/>
-<wire x1="340.36" y1="173.99" x2="346.71" y2="173.99" width="0.1524" layer="91"/>
-<junction x="340.36" y="173.99"/>
-</segment>
-</net>
-<net name="N$5" class="0">
+<wire x1="336.55" y1="173.99" x2="346.71" y2="173.99" width="0.1524" layer="91"/>
+<junction x="336.55" y="173.99"/>
+<label x="337.82" y="173.99" size="1.778" layer="95"/>
+</segment>
+</net>
+<net name="IN3" class="0">
 <segment>
 <pinref part="U1" gate="G$1" pin="IO18"/>
 <wire x1="252.73" y1="177.8" x2="325.12" y2="177.8" width="0.1524" layer="91"/>
 <pinref part="U$1" gate="G$1" pin="IN3"/>
-<wire x1="346.71" y1="176.53" x2="340.36" y2="176.53" width="0.1524" layer="91"/>
-<wire x1="340.36" y1="176.53" x2="325.12" y2="176.53" width="0.1524" layer="91"/>
+<wire x1="346.71" y1="176.53" x2="336.55" y2="176.53" width="0.1524" layer="91"/>
+<wire x1="336.55" y1="176.53" x2="325.12" y2="176.53" width="0.1524" layer="91"/>
 <wire x1="325.12" y1="176.53" x2="325.12" y2="177.8" width="0.1524" layer="91"/>
 <pinref part="U$7" gate="G$1" pin="3"/>
-<junction x="340.36" y="176.53"/>
+<junction x="336.55" y="176.53"/>
+<label x="337.82" y="176.53" size="1.778" layer="95"/>
 </segment>
 </net>
@@
 </segment>
 </net>
-<net name="N$6" class="0">
+<net name="IN8" class="0">
 <segment>
 <pinref part="U1" gate="G$1" pin="IO15"/>
@@
 <wire x1="320.04" y1="160.02" x2="320.04" y2="163.83" width="0.1524" layer="91"/>
 <pinref part="U$1" gate="G$1" pin="IN8"/>
-<wire x1="320.04" y1="163.83" x2="340.36" y2="163.83" width="0.1524" layer="91"/>
+<wire x1="320.04" y1="163.83" x2="336.55" y2="163.83" width="0.1524" layer="91"/>
 <pinref part="U$7" gate="G$1" pin="8"/>
-<wire x1="340.36" y1="163.83" x2="346.71" y2="163.83" width="0.1524" layer="91"/>
-<junction x="340.36" y="163.83"/>
-</segment>
-</net>
-<net name="N$7" class="0">
+<wire x1="336.55" y1="163.83" x2="346.71" y2="163.83" width="0.1524" layer="91"/>
+<junction x="336.55" y="163.83"/>
+<label x="337.82" y="163.83" size="1.778" layer="95"/>
+</segment>
+</net>
+<net name="IN7" class="0">
 <segment>
 <pinref part="U$1" gate="G$1" pin="IN7"/>
-<wire x1="317.5" y1="166.37" x2="340.36" y2="166.37" width="0.1524" layer="91"/>
-<wire x1="340.36" y1="166.37" x2="346.71" y2="166.37" width="0.1524" layer="91"/>
+<wire x1="317.5" y1="166.37" x2="336.55" y2="166.37" width="0.1524" layer="91"/>
+<wire x1="336.55" y1="166.37" x2="346.71" y2="166.37" width="0.1524" layer="91"/>
 <wire x1="317.5" y1="166.37" x2="317.5" y2="144.78" width="0.1524" layer="91"/>
 <wire x1="317.5" y1="144.78" x2="228.6" y2="144.78" width="0.1524" layer="91"/>
@@
 <wire x1="228.6" y1="162.56" x2="212.09" y2="162.56" width="0.1524" layer="91"/>
 <pinref part="U$7" gate="G$1" pin="7"/>
-<junction x="340.36" y="166.37"/>
-</segment>
-</net>
-<net name="N$8" class="0">
+<junction x="336.55" y="166.37"/>
+<label x="337.82" y="166.37" size="1.778" layer="95"/>
+</segment>
+</net>
+<net name="IN2" class="0">
 <segment>
 <pinref part="U1" gate="G$1" pin="IO19"/>
@@
 <pinref part="U$1" gate="G$1" pin="IN2"/>
 <wire x1="327.66" y1="180.34" x2="327.66" y2="179.07" width="0.1524" layer="91"/>
-<wire x1="327.66" y1="179.07" x2="340.36" y2="179.07" width="0.1524" layer="91"/>
+<wire x1="327.66" y1="179.07" x2="336.55" y2="179.07" width="0.1524" layer="91"/>
 <pinref part="U$7" gate="G$1" pin="2"/>
-<wire x1="340.36" y1="179.07" x2="346.71" y2="179.07" width="0.1524" layer="91"/>
-<junction x="340.36" y="179.07"/>
-</segment>
-</net>
-<net name="N$9" class="0">
+<wire x1="336.55" y1="179.07" x2="346.71" y2="179.07" width="0.1524" layer="91"/>
+<junction x="336.55" y="179.07"/>
+<label x="337.82" y="179.07" size="1.778" layer="95"/>
+</segment>
+</net>
+<net name="IN1" class="0">
 <segment>
 <pinref part="U1" gate="G$1" pin="IO23"/>
@@
 <pinref part="U$1" gate="G$1" pin="IN1"/>
 <wire x1="302.26" y1="195.58" x2="302.26" y2="181.61" width="0.1524" layer="91"/>
-<wire x1="302.26" y1="181.61" x2="340.36" y2="181.61" width="0.1524" layer="91"/>
+<wire x1="302.26" y1="181.61" x2="336.55" y2="181.61" width="0.1524" layer="91"/>
 <pinref part="U$7" gate="G$1" pin="1"/>
-<wire x1="340.36" y1="181.61" x2="346.71" y2="181.61" width="0.1524" layer="91"/>
-<junction x="340.36" y="181.61"/>
+<wire x1="336.55" y1="181.61" x2="346.71" y2="181.61" width="0.1524" layer="91"/>
+<junction x="336.55" y="181.61"/>
+<label x="337.82" y="181.61" size="1.778" layer="95"/>
 </segment>
 </net>
@@
 </segment>
 </net>
-<net name="N$13" class="0">
+<net name="DS18B20" class="0">
 <segment>
 <pinref part="U$6" gate="G$1" pin="4"/>
@@
 <pinref part="R1" gate="G$1" pin="1"/>
 <junction x="149.86" y="177.8"/>
-</segment>
-</net>
-<net name="N$10" class="0">
+<label x="201.93" y="182.88" size="1.778" layer="95"/>
+</segment>
+</net>
+<net name="REED_2" class="0">
 <segment>
 <pinref part="S1" gate="G$1" pin="1"/>
@@
 <wire x1="144.78" y1="172.72" x2="212.09" y2="172.72" width="0.1524" layer="91"/>
 <junction x="144.78" y="172.72"/>
-</segment>
-</net>
-<net name="N$14" class="0">
+<label x="198.12" y="172.72" size="1.778" layer="95"/>
+</segment>
+</net>
+<net name="REED_1" class="0">
 <segment>
 <pinref part="S2" gate="G$1" pin="1"/>
@@
 <pinref part="U1" gate="G$1" pin="IO14"/>
 <wire x1="198.12" y1="170.18" x2="212.09" y2="170.18" width="0.1524" layer="91"/>
-</segment>
-</net>
-<net name="N$11" class="0">
+<label x="198.12" y="170.18" size="1.778" layer="95"/>
+</segment>
+</net>
+<net name="BUZZER" class="0">
 <segment>
 <pinref part="SG1" gate="G$1" pin="1"/>
@@
 <wire x1="200.66" y1="256.54" x2="200.66" y2="175.26" width="0.1524" layer="91"/>
 <junction x="274.32" y="256.54"/>
-</segment>
-</net>
-<net name="N$2" class="0">
+<label x="201.93" y="175.26" size="1.778" layer="95"/>
+</segment>
+</net>
+<net name="IN6" class="0">
 <segment>
 <pinref part="U$1" gate="G$1" pin="IN6"/>
-<wire x1="346.71" y1="168.91" x2="340.36" y2="168.91" width="0.1524" layer="91"/>
-<wire x1="340.36" y1="168.91" x2="314.96" y2="168.91" width="0.1524" layer="91"/>
+<wire x1="346.71" y1="168.91" x2="336.55" y2="168.91" width="0.1524" layer="91"/>
+<wire x1="336.55" y1="168.91" x2="314.96" y2="168.91" width="0.1524" layer="91"/>
 <wire x1="314.96" y1="168.91" x2="314.96" y2="147.32" width="0.1524" layer="91"/>
 <wire x1="314.96" y1="147.32" x2="231.14" y2="147.32" width="0.1524" layer="91"/>
@@
 <wire x1="231.14" y1="177.8" x2="212.09" y2="177.8" width="0.1524" layer="91"/>
 <pinref part="U$7" gate="G$1" pin="6"/>
-<junction x="340.36" y="168.91"/>
-</segment>
-</net>
+<junction x="336.55" y="168.91"/>
+<label x="337.82" y="168.91" size="1.778" layer="95"/>
+</segment>
+</net>
