File: Hardware/Nodeboard/Routing versions/OECOC_controlbordroutes.brd (EAGLE design)
At the start: 100 x 65 mm, 10 parts, among them U1 ESP32-DEVKITC-32D

Commit message: further pcb development
Parts:
- added U$1: (no value), Personal:LOGO
- added U$10: (no value), Personal:LOGO_PHOENIX-CONTACT
- added U$2, U$4: (no value), micro-philips:I2C
- added U$5: (no value), Personal:LOGO_EXO-TERRA
- added U$9: (no value), Personal:LOGO_ESPRESSIF-SYSTEMS
- R1: value (none) -> 4k7
Connections:
- removed net 3V3: U1.1
- net +3V3: now also U1.1
Routing:
- net IN1: track 0.00 -> 73.1 mm, vias 0 -> 1
- net +3V3: track 0.00 -> 72.9 mm
- net IN2: track 0.00 -> 61.0 mm
- net SCL: track 0.00 -> 59.7 mm
- net SDA: track 0.00 -> 59.3 mm
- net REED_1: track 0.00 -> 58.2 mm, vias 0 -> 1
- net +5V: track 0.00 -> 53.1 mm
- net REED_2: track 0.00 -> 53.1 mm, vias 0 -> 1
- net IN6: track 0.00 -> 51.2 mm, vias 0 -> 1
- net IN3: track 0.00 -> 49.8 mm, vias 0 -> 1
- net IN4: track 0.00 -> 43.8 mm, vias 0 -> 1
- net BUZZER: track 0.00 -> 42.8 mm
- net DS18B20: track 0.00 -> 41.7 mm
- net IN7: track 0.00 -> 40.6 mm, vias 0 -> 1
- net IN5: track 0.00 -> 39.6 mm
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Other:
- board text added: "Design: Nathan Laureyn Date: 11/10/2021 Ver: 1"
